File: firstProto/kicad/ampStation.sch (KiCad schematic (older format))
At the start: 13 parts, among them J1 Conn_01x02, J2 Conn_01x02, J3 Conn_01x02, U1 TL072, U2 MAX1044

Commit message: misc
Parts:
- U1: value TL072 -> LM348D; Spice_Lib_File (none) -> /Volumes/SSD/Dev/_Electronique/ampStation/Kicad-libs/LM348.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; Spice_Model (none) -> LM348; Spice_Netlist_Enabled (none) -> Y; Spice_Node_Sequence (none) -> 3 2 8 4 1; Spice_Primitive (none) -> X
- U2: Spice_Lib_File (none) -> /Volumes/SSD/Dev/_Electronique/ampStation/Kicad-libs/TL072.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; Spice_Model (none) -> TL072; Spice_Netlist_Enabled (none) -> N; Spice_Primitive (none) -> X
Connections:
- net VCC: now reaches J3.1 (Pin_1), R3.1, U1.8 (V+), U2.8 (V+)
Other:
- note added: "* Alimentation 5V"
- note added: "* Entrée du signal"
- note added: "* Sortie vers microcontroleur"
- note added: "- Les résistances R1 et R2 doivent être ajustées\n en fonction du gain désiré\n- Les résistances R3 et R4 doivent être ajustées\n en fonction de l'OFFSET désiré.\n- On doit donc avoir des supports pour ces \n 4 résistances (et non les souder sur la plaque de prototypage)"
- moved on the sheet: C2, C3, J3, U1C, U2
Changed lines of the file:
@@
 P 4600 1600
 F 0 "U1" H 4600 1967 50  0000 C CNN
-F 1 "TL072" H 4600 1876 50  0000 C CNN
+F 1 "LM348D" H 4600 1876 50  0000 C CNN
 F 2 "" H 4600 1600 50  0001 C CNN
 F 3 "http://www.ti.com/lit/ds/symlink/tl071.pdf" H 4600 1600 50  0001 C CNN
+F 4 "X" H 4600 1600 50  0001 C CNN "Spice_Primitive"
+F 5 "LM348" H 4600 1600 50  0001 C CNN "Spice_Model"
+F 6 "Y" H 4600 1600 50  0001 C CNN "Spice_Netlist_Enabled"
+F 7 "/Volumes/SSD/Dev/_Electronique/ampStation/Kicad-libs/LM348.lib" H 4600 1600 50  0001 C CNN "Spice_Lib_File"
+F 8 "3 2 8 4 1" H 4600 1600 50  0001 C CNN "Spice_Node_Sequence"
 	1    4600 1600
 	1    0    0    -1
@@
 L Regulator_SwitchedCapacitor:MAX1044 U2
 U 1 1 605C67EF
-P 6000 4000
-F 0 "U2" H 6000 4567 50  0000 C CNN
-F 1 "MAX1044" H 6000 4476 50  0000 C CNN
-F 2 "" H 6100 3900 50  0001 C CNN
-F 3 "http://datasheets.maximintegrated.com/en/ds/ICL7660-MAX1044.pdf" H 6100 3900 50  0001 C CNN
-	1    6000 4000
+P 4400 3800
+F 0 "U2" H 4400 4367 50  0000 C CNN
+F 1 "MAX1044" H 4400 4276 50  0000 C CNN
+F 2 "" H 4500 3700 50  0001 C CNN
+F 3 "http://datasheets.maximintegrated.com/en/ds/ICL7660-MAX1044.pdf" H 4500 3700 50  0001 C CNN
+F 4 "X" H 4400 3800 50  0001 C CNN "Spice_Primitive"
+F 5 "TL072" H 4400 3800 50  0001 C CNN "Spice_Model"
+F 6 "N" H 4400 3800 50  0001 C CNN "Spice_Netlist_Enabled"
+F 7 "/Volumes/SSD/Dev/_Electronique/ampStation/Kicad-libs/TL072.lib" H 4400 3800 50  0001 C CNN "Spice_Lib_File"
+	1    4400 3800
 	1    0    0    -1
 $EndComp
@@
 L Device:CP C3
 U 1 1 605C96CB
-P 6650 4100
-F 0 "C3" H 6768 4146 50  0000 L CNN
-F 1 "10u" H 6768 4055 50  0000 L CNN
-F 2 "" H 6688 3950 50  0001 C CNN
-F 3 "~" H 6650 4100 50  0001 C CNN
-	1    6650 4100
+P 5050 3900
+F 0 "C3" H 5168 3946 50  0000 L CNN
+F 1 "10u" H 5168 3855 50  0000 L CNN
+F 2 "" H 5088 3750 50  0001 C CNN
+F 3 "~" H 5050 3900 50  0001 C CNN
+	1    5050 3900
 	1    0    0    -1
 $EndComp
@@
 L Device:CP C2
 U 1 1 605CF0F7
-P 6500 3500
-F 0 "C2" H 6618 3546 50  0000 L CNN
-F 1 "10u" H 6618 3455 50  0000 L CNN
-F 2 "" H 6538 3350 50  0001 C CNN
-F 3 "~" H 6500 3500 50  0001 C CNN
-	1    6500 3500
+P 4900 3300
+F 0 "C2" H 5018 3346 50  0000 L CNN
+F 1 "10u" H 5018 3255 50  0000 L CNN
+F 2 "" H 4938 3150 50  0001 C CNN
+F 3 "~" H 4900 3300 50  0001 C CNN
+	1    4900 3300
 	1    0    0    -1
 $EndComp
@@
 L Amplifier_Operational:TL072 U1
 U 3 1 605F9529
-P 7200 3300
-F 0 "U1" H 7158 3346 50  0000 L CNN
-F 1 "TL072" H 7158 3255 50  0000 L CNN
-F 2 "" H 7200 3300 50  0001 C CNN
-F 3 "http://www.ti.com/lit/ds/symlink/tl071.pdf" H 7200 3300 50  0001 C CNN
-	3    7200 3300
-	1    0    0    -1
-$EndComp
-Wire Wire Line
-	5300 3700 5600 3700
-Wire Wire Line
-	6400 3900 6650 3900
-Wire Wire Line
-	6650 3900 6650 3950
-Wire Wire Line
-	6400 4300 6650 4300
-Wire Wire Line
-	6650 4300 6650 4250
+P 5600 3100
+F 0 "U1" H 5558 3146 50  0000 L CNN
+F 1 "TL072" H 5558 3055 50  0000 L CNN
+F 2 "" H 5600 3100 50  0001 C CNN
+F 3 "http://www.ti.com/lit/ds/symlink/tl071.pdf" H 5600 3100 50  0001 C CNN
+	3    5600 3100
+	1    0    0    -1
+$EndComp
+Wire Wire Line
+	4800 3700 5050 3700
+Wire Wire Line
+	5050 3700 5050 3750
+Wire Wire Line
+	4800 4100 5050 4100
+Wire Wire Line
+	5050 4100 5050 4050
 $Comp
 L power:GND #PWR07
 U 1 1 60603A06
-P 6850 3200
-F 0 "#PWR07" H 6850 2950 50  0001 C CNN
-F 1 "GND" H 6855 3027 50  0000 C CNN
-F 2 "" H 6850 3200 50  0001 C CNN
-F 3 "" H 6850 3200 50  0001 C CNN
-	1    6850 3200
-	1    0    0    -1
-$EndComp
-Wire Wire Line
-	6400 3700 6500 3700
-Wire Wire Line
-	6500 3700 6500 3650
-Wire Wire Line
-	6500 3700 7100 3700
-Wire Wire Line
-	7100 3700 7100 3600
-Connection ~ 6500 3700
-Wire Wire Line
-	6500 3350 6500 3150
-Wire Wire Line
-	6500 3150 6850 3150
-Wire Wire Line
-	6850 3150 6850 3200
+P 5250 3000
+F 0 "#PWR07" H 5250 2750 50  0001 C CNN
+F 1 "GND" H 5255 2827 50  0000 C CNN
+F 2 "" H 5250 3000 50  0001 C CNN
+F 3 "" H 5250 3000 50  0001 C CNN
+	1    5250 3000
+	1    0    0    -1
+$EndComp
+Wire Wire Line
+	4800 3500 4900 3500
+Wire Wire Line
+	4900 3500 4900 3450
+Wire Wire Line
+	4900 3500 5500 3500
+Wire Wire Line
+	5500 3500 5500 3400
+Connection ~ 4900 3500
+Wire Wire Line
+	4900 3150 4900 2950
+Wire Wire Line
+	4900 2950 5250 2950
+Wire Wire Line
+	5250 2950 5250 3000
 $Comp
 L power:GND #PWR06
 U 1 1 60607759
-P 6000 4600
-F 0 "#PWR06" H 6000 4350 50  0001 C CNN
-F 1 "GND" H 6005 4427 50  0000 C CNN
-F 2 "" H 6000 4600 50  0001 C CNN
-F 3 "" H 6000 4600 50  0001 C CNN
-	1    6000 4600
-	1    0    0    -1
-$EndComp
-Wire Wire Line
-	7100 3000 7100 2900
+P 4400 4400
+F 0 "#PWR06" H 4400 4150 50  0001 C CNN
+F 1 "GND" H 4405 4227 50  0000 C CNN
+F 2 "" H 4400 4400 50  0001 C CNN
+F 3 "" H 4400 4400 50  0001 C CNN
+	1    4400 4400
+	1    0    0    -1
+$EndComp
 $Comp
 L Device:CP C1
@@
 Wire Wire Line
 	6500 2000 6500 2100
-NoConn ~ 5600 4000
-NoConn ~ 5600 4200
-Wire Wire Line
-	6000 4500 6000 4600
+NoConn ~ 4000 3800
+NoConn ~ 4000 4000
+Wire Wire Line
+	4400 4300 4400 4400
 $Comp
 L Device:CP C4
@@
 L Connector_Generic:Conn_01x02 J3
 U 1 1 605DDC07
-P 8250 2350
-F 0 "J3" H 8168 2567 50  0000 C CNN
-F 1 "Conn_01x02" H 8168 2476 50  0000 C CNN
-F 2 "" H 8250 2350 50  0001 C CNN
-F 3 "~" H 8250 2350 50  0001 C CNN
-F 4 "I" H 8250 2350 50  0001 C CNN "Spice_Primitive"
-F 5 "dc 5" H 8250 2350 50  0001 C CNN "Spice_Model"
-F 6 "Y" H 8250 2350 50  0001 C CNN "Spice_Netlist_Enabled"
-	1    8250 2350
+P 3200 3500
+F 0 "J3" H 3118 3717 50  0000 C CNN
+F 1 "Conn_01x02" H 3118 3626 50  0000 C CNN
+F 2 "" H 3200 3500 50  0001 C CNN
+F 3 "~" H 3200 3500 50  0001 C CNN
+F 4 "I" H 3200 3500 50  0001 C CNN "Spice_Primitive"
+F 5 "dc 5" H 3200 3500 50  0001 C CNN "Spice_Model"
+F 6 "Y" H 3200 3500 50  0001 C CNN "Spice_Netlist_Enabled"
+	1    3200 3500
 	-1   0    0    -1
 $EndComp
@@
 L power:GND #PWR012
 U 1 1 605DF297
-P 8800 2550
-F 0 "#PWR012" H 8800 2300 50  0001 C CNN
-F 1 "GND" H 8805 2377 50  0000 C CNN
-F 2 "" H 8800 2550 50  0001 C CNN
-F 3 "" H 8800 2550 50  0001 C CNN
-	1    8800 2550
-	1    0    0    -1
-$EndComp
-Wire Wire Line
-	8450 2450 8800 2450
-Wire Wire Line
-	8800 2450 8800 2550
-Wire Wire Line
-	8800 2350 8450 2350
-Wire Wire Line
-	8800 2350 8800 1900
-Wire Wire Line
-	8800 950  6500 950
-Wire Wire Line
-	6500 950  6500 1200
-Wire Wire Line
-	8800 1900 7700 1900
-Wire Wire Line
-	7700 1900 7700 2900
-Wire Wire Line
-	7700 2900 7100 2900
-Connection ~ 8800 1900
-Wire Wire Line
-	8800 1900 8800 950
-Wire Wire Line
-	7100 2900 5300 2900
-Wire Wire Line
-	5300 2900 5300 3700
-Connection ~ 7100 2900
+P 3750 3750
+F 0 "#PWR012" H 3750 3500 50  0001 C CNN
+F 1 "GND" H 3755 3577 50  0000 C CNN
+F 2 "" H 3750 3750 50  0001 C CNN
+F 3 "" H 3750 3750 50  0001 C CNN
+	1    3750 3750
+	1    0    0    -1
+$EndComp
+Wire Wire Line
+	3400 3600 3750 3600
+Text Notes 2900 1350 0    50   ~ 0
+* Entrée du signal
+Wire Wire Line
+	3750 3750 3750 3600
+$Comp
+L power:VCC #PWR?
+U 1 1 60602642
+P 3750 3200
+F 0 "#PWR?" H 3750 3050 50  0001 C CNN
+F 1 "VCC" H 3767 3373 50  0000 C CNN
+F 2 "" H 3750 3200 50  0001 C CNN
+F 3 "" H 3750 3200 50  0001 C CNN
+	1    3750 3200
+	1    0    0    -1
+$EndComp
+$Comp
+L power:VCC #PWR?
+U 1 1 60602D61
+P 5500 2600
+F 0 "#PWR?" H 5500 2450 50  0001 C CNN
+F 1 "VCC" H 5517 2773 50  0000 C CNN
+F 2 "" H 5500 2600 50  0001 C CNN
+F 3 "" H 5500 2600 50  0001 C CNN
+	1    5500 2600
+	1    0    0    -1
+$EndComp
+Wire Wire Line
+	3400 3500 3750 3500
+Wire Wire Line
+	3750 3500 3750 3200
+Connection ~ 3750 3500
+Wire Wire Line
+	3750 3500 4000 3500
+Wire Wire Line
+	5500 2600 5500 2800
+$Comp
+L power:VCC #PWR?
+U 1 1 6060556A
+P 6500 1000
+F 0 "#PWR?" H 6500 850 50  0001 C CNN
+F 1 "VCC" H 6517 1173 50  0000 C CNN
+F 2 "" H 6500 1000 50  0001 C CNN
+F 3 "" H 6500 1000 50  0001 C CNN
+	1    6500 1000
+	1    0    0    -1
+$EndComp
+Wire Wire Line
+	6500 1200 6500 1000
+Text Notes 2850 3150 0    50   ~ 0
+* Alimentation 5V
+Text Notes 7050 1450 0    50   ~ 0
+* Sortie vers microcontroleur
+Text Notes 6250 3650 0    50   ~ 0
+- Les résistances R1 et R2 doivent être ajustées\n   en fonction du gain désiré\n- Les résistances R3 et R4 doivent être ajustées\n   en fonction de l'OFFSET désiré.\n- On doit donc avoir des supports pour ces \n   4 résistances (et non les souder sur la plaque de prototypage)
 $EndSCHEMATC

Commit message: misc
Parts:
- removed R2, R4: 10k, symbol Device:R
- added RV1: 10k, Connector_PinSocket_2.54mm:PinSocket_1x03_P2.54mm_Vertical, symbol Device:R_POT_US
- added RV2: 100k, Connector_PinSocket_2.54mm:PinSocket_1x03_P2.54mm_Vertical, symbol Device:R_POT_US
- C1, C3: footprint (none) -> Capacitor_THT:C_Axial_L17.0mm_D7.0mm_P20.00mm_Horizontal
- C2: renamed from C4; footprint (none) -> Capacitor_THT:C_Axial_L17.0mm_D7.0mm_P20.00mm_Horizontal
- C4: renamed from C2; footprint (none) -> Capacitor_THT:C_Axial_L17.0mm_D7.0mm_P20.00mm_Horizontal
- J1, J2: footprint (none) -> EH_Modules:Bornier_2pts_L10mm_W9mm_P5mm
- J3: value Conn_01x02 -> Alim5V; footprint (none) -> EH_Modules:Bornier_2pts_L10mm_W9mm_P5mm
- R1: footprint (none) -> Connector_PinSocket_2.54mm:PinSocket_1x06_P2.54mm_Vertical
- R2: renamed from R3; footprint (none) -> Connector_PinSocket_2.54mm:PinSocket_1x06_P2.54mm_Vertical
- U1: footprint (none) -> Package_DIP:DIP-14_W7.62mm
- U1: value TL072 -> LM348D; footprint (none) -> Package_DIP:DIP-14_W7.62mm
- U2: footprint (none) -> Package_DIP:DIP-8_W7.62mm
Connections:
- net GND: now also RV2.1, RV2.2
- net at C1.1, C2.1, U1.1: now also RV1.1, RV1.2
- net at R1.1, U1.2 (-): now also RV1.3
- net at C2.2, J2.1 (Pin_1), R2.2: now also RV2.3
Other:
- note added: "- Les résistances RV1 et RV2 sont ajustées\n en fonction du gain et de l'OFFSET désirés\n- supports pour R1, R3, RV1 et RV2"
- note removed: "- Les résistances R1 et R2 doivent être ajustées\n en fonction du gain désiré\n- Les résistances R3 et R4 doivent être ajustées\n en fonction de l'OFFSET désiré.\n- On doit donc avoir des supports pour ces \n 4 résistances (et non les souder sur la plaque de prototypage)"
Changed lines of the file:
@@
 F 0 "U1" H 4600 1967 50  0000 C CNN
 F 1 "LM348D" H 4600 1876 50  0000 C CNN
-F 2 "" H 4600 1600 50  0001 C CNN
-F 3 "http://www.ti.com/lit/ds/symlink/tl071.pdf" H 4600 1600 50  0001 C CNN
+F 2 "Package_DIP:DIP-14_W7.62mm" H 4600 1600 50  0001 C CNN
+F 3 "" H 4600 1600 50  0001 C CNN
 F 4 "X" H 4600 1600 50  0001 C CNN "Spice_Primitive"
 F 5 "LM348" H 4600 1600 50  0001 C CNN "Spice_Model"
@@
 $EndComp
 $Comp
-L Device:R R2
-U 1 1 605BAC0A
-P 4600 2150
-F 0 "R2" V 4807 2150 50  0000 C CNN
-F 1 "10k" V 4716 2150 50  0000 C CNN
-F 2 "" V 4530 2150 50  0001 C CNN
-F 3 "~" H 4600 2150 50  0001 C CNN
-	1    4600 2150
-	0    -1   -1   0
-$EndComp
-$Comp
 L Device:R R1
 U 1 1 605BB7B2
@@
 F 0 "R1" V 3643 1700 50  0000 C CNN
 F 1 "1k" V 3734 1700 50  0000 C CNN
-F 2 "" V 3780 1700 50  0001 C CNN
+F 2 "Connector_PinSocket_2.54mm:PinSocket_1x06_P2.54mm_Vertical" V 3780 1700 50  0001 C CNN
 F 3 "~" H 3850 1700 50  0001 C CNN
 	1    3850 1700
@@
 F 0 "U2" H 4400 4367 50  0000 C CNN
 F 1 "MAX1044" H 4400 4276 50  0000 C CNN
-F 2 "" H 4500 3700 50  0001 C CNN
+F 2 "Package_DIP:DIP-8_W7.62mm" H 4500 3700 50  0001 C CNN
 F 3 "http://datasheets.maximintegrated.com/en/ds/ICL7660-MAX1044.pdf" H 4500 3700 50  0001 C CNN
 F 4 "X" H 4400 3800 50  0001 C CNN "Spice_Primitive"
@@
 F 0 "C3" H 5168 3946 50  0000 L CNN
 F 1 "10u" H 5168 3855 50  0000 L CNN
-F 2 "" H 5088 3750 50  0001 C CNN
+F 2 "Capacitor_THT:C_Axial_L17.0mm_D7.0mm_P20.00mm_Horizontal" H 5088 3750 50  0001 C CNN
 F 3 "~" H 5050 3900 50  0001 C CNN
 	1    5050 3900
@@
 $EndComp
 $Comp
-L Device:CP C2
+L Device:CP C4
 U 1 1 605CF0F7
 P 4900 3300
-F 0 "C2" H 5018 3346 50  0000 L CNN
+F 0 "C4" H 5018 3346 50  0000 L CNN
 F 1 "10u" H 5018 3255 50  0000 L CNN
-F 2 "" H 4938 3150 50  0001 C CNN
+F 2 "Capacitor_THT:C_Axial_L17.0mm_D7.0mm_P20.00mm_Horizontal" H 4938 3150 50  0001 C CNN
 F 3 "~" H 4900 3300 50  0001 C CNN
 	1    4900 3300
@@
 P 5600 3100
 F 0 "U1" H 5558 3146 50  0000 L CNN
-F 1 "TL072" H 5558 3055 50  0000 L CNN
-F 2 "" H 5600 3100 50  0001 C CNN
+F 1 "LM348D" H 5558 3055 50  0000 L CNN
+F 2 "Package_DIP:DIP-14_W7.62mm" H 5600 3100 50  0001 C CNN
 F 3 "http://www.ti.com/lit/ds/symlink/tl071.pdf" H 5600 3100 50  0001 C CNN
 	3    5600 3100
@@
 F 0 "C1" H 5468 1896 50  0000 L CNN
 F 1 "10u" H 5468 1805 50  0000 L CNN
-F 2 "" H 5388 1700 50  0001 C CNN
+F 2 "Capacitor_THT:C_Axial_L17.0mm_D7.0mm_P20.00mm_Horizontal" H 5388 1700 50  0001 C CNN
 F 3 "~" H 5350 1850 50  0001 C CNN
 	1    5350 1850
@@
 $EndComp
 $Comp
-L Device:R R3
+L Device:R R2
 U 1 1 606343F6
 P 6500 1350
-F 0 "R3" H 6570 1396 50  0000 L CNN
+F 0 "R2" H 6570 1396 50  0000 L CNN
 F 1 "10k" H 6570 1305 50  0000 L CNN
-F 2 "" V 6430 1350 50  0001 C CNN
+F 2 "Connector_PinSocket_2.54mm:PinSocket_1x06_P2.54mm_Vertical" V 6430 1350 50  0001 C CNN
 F 3 "~" H 6500 1350 50  0001 C CNN
 	1    6500 1350
-	1    0    0    -1
-$EndComp
-$Comp
-L Device:R R4
-U 1 1 60634BE6
-P 6500 1850
-F 0 "R4" H 6570 1896 50  0000 L CNN
-F 1 "10k" H 6570 1805 50  0000 L CNN
-F 2 "" V 6430 1850 50  0001 C CNN
-F 3 "~" H 6500 1850 50  0001 C CNN
-	1    6500 1850
 	1    0    0    -1
 $EndComp
@@
 Connection ~ 6500 1600
 Wire Wire Line
-	6500 2000 6500 2100
+	6500 2000 6500 2050
 NoConn ~ 4000 3800
 NoConn ~ 4000 4000
@@
 	4400 4300 4400 4400
 $Comp
-L Device:CP C4
+L Device:CP C2
 U 1 1 60611391
 P 5950 1600
-F 0 "C4" V 6100 1650 50  0000 L CNN
+F 0 "C2" V 6100 1650 50  0000 L CNN
 F 1 "10u" V 5750 1550 50  0000 L CNN
-F 2 "" H 5988 1450 50  0001 C CNN
+F 2 "Capacitor_THT:C_Axial_L17.0mm_D7.0mm_P20.00mm_Horizontal" H 5988 1450 50  0001 C CNN
 F 3 "~" H 5950 1600 50  0001 C CNN
 	1    5950 1600
@@
 F 0 "J1" H 2818 1917 50  0000 C CNN
 F 1 "Conn_01x02" H 2818 1826 50  0000 C CNN
-F 2 "" H 2900 1700 50  0001 C CNN
+F 2 "EH_Modules:Bornier_2pts_L10mm_W9mm_P5mm" H 2900 1700 50  0001 C CNN
 F 3 "~" H 2900 1700 50  0001 C CNN
 F 4 "V" H 2900 1700 50  0001 C CNN "Spice_Primitive"
@@
 F 0 "J2" H 7330 1592 50  0000 L CNN
 F 1 "Conn_01x02" H 7330 1501 50  0000 L CNN
-F 2 "" H 7250 1600 50  0001 C CNN
+F 2 "EH_Modules:Bornier_2pts_L10mm_W9mm_P5mm" H 7250 1600 50  0001 C CNN
 F 3 "~" H 7250 1600 50  0001 C CNN
 F 4 "I" H 7250 1600 50  0001 C CNN "Spice_Primitive"
@@
 P 3200 3500
 F 0 "J3" H 3118 3717 50  0000 C CNN
-F 1 "Conn_01x02" H 3118 3626 50  0000 C CNN
-F 2 "" H 3200 3500 50  0001 C CNN
+F 1 "Alim5V" H 3118 3626 50  0000 C CNN
+F 2 "EH_Modules:Bornier_2pts_L10mm_W9mm_P5mm" H 3200 3500 50  0001 C CNN
 F 3 "~" H 3200 3500 50  0001 C CNN
 F 4 "I" H 3200 3500 50  0001 C CNN "Spice_Primitive"
@@
 	3750 3750 3750 3600
 $Comp
-L power:VCC #PWR?
+L power:VCC #PWR03
 U 1 1 60602642
 P 3750 3200
-F 0 "#PWR?" H 3750 3050 50  0001 C CNN
+F 0 "#PWR03" H 3750 3050 50  0001 C CNN
 F 1 "VCC" H 3767 3373 50  0000 C CNN
 F 2 "" H 3750 3200 50  0001 C CNN
@@
 $EndComp
 $Comp
-L power:VCC #PWR?
+L power:VCC #PWR05
 U 1 1 60602D61
 P 5500 2600
-F 0 "#PWR?" H 5500 2450 50  0001 C CNN
+F 0 "#PWR05" H 5500 2450 50  0001 C CNN
 F 1 "VCC" H 5517 2773 50  0000 C CNN
 F 2 "" H 5500 2600 50  0001 C CNN
@@
 	5500 2600 5500 2800
 $Comp
-L power:VCC #PWR?
+L power:VCC #PWR08
 U 1 1 6060556A
 P 6500 1000
-F 0 "#PWR?" H 6500 850 50  0001 C CNN
+F 0 "#PWR08" H 6500 850 50  0001 C CNN
 F 1 "VCC" H 6517 1173 50  0000 C CNN
 F 2 "" H 6500 1000 50  0001 C CNN
@@
 * Sortie vers microcontroleur
 Text Notes 6250 3650 0    50   ~ 0
-- Les résistances R1 et R2 doivent être ajustées\n   en fonction du gain désiré\n- Les résistances R3 et R4 doivent être ajustées\n   en fonction de l'OFFSET désiré.\n- On doit donc avoir des supports pour ces \n   4 résistances (et non les souder sur la plaque de prototypage)
+- Les résistances RV1 et RV2 sont ajustées\n   en fonction du gain et de l'OFFSET désirés\n- supports pour R1, R3, RV1 et RV2
+$Comp
+L Device:R_POT_US RV1
+U 1 1 605FC834
+P 4600 2150
+F 0 "RV1" V 4395 2150 50  0000 C CNN
+F 1 "10k" V 4486 2150 50  0000 C CNN
+F 2 "Connector_PinSocket_2.54mm:PinSocket_1x03_P2.54mm_Vertical" H 4600 2150 50  0001 C CNN
+F 3 "~" H 4600 2150 50  0001 C CNN
+	1    4600 2150
+	0    1    1    0
+$EndComp
+Wire Wire Line
+	4600 2300 4600 2400
+Wire Wire Line
+	4600 2400 5100 2400
+Wire Wire Line
+	5100 2400 5100 2150
+Connection ~ 5100 2150
+$Comp
+L Device:R_POT_US RV2
+U 1 1 605FFC42
+P 6500 1850
+F 0 "RV2" H 6432 1804 50  0000 R CNN
+F 1 "100k" H 6432 1895 50  0000 R CNN
+F 2 "Connector_PinSocket_2.54mm:PinSocket_1x03_P2.54mm_Vertical" H 6500 1850 50  0001 C CNN
+F 3 "~" H 6500 1850 50  0001 C CNN
+	1    6500 1850
+	-1   0    0    1
+$EndComp
+Wire Wire Line
+	6350 1850 6350 2050
+Wire Wire Line
+	6350 2050 6500 2050
+Connection ~ 6500 2050
+Wire Wire Line
+	6500 2050 6500 2100
 $EndSCHEMATC
