File: firstProto/kicad/ampStation.kicad_pcb (KiCad board)
At the start: 2 copper layers, 150 x 50 mm, 13 parts, among them J1 Conn_01x02, J2 Conn_01x02, J3 Conn_01x02, U1 LM348D, U2 MAX1044

Commit message: misc
Parts:
- moved U2 111.7 mm to (149.9, 113.0), turned to 90 degrees
- moved J1 47.3 mm to (40.6, 99.1), turned to 180 degrees
Routing:
- net (no net): track 0.00 -> 2199.6 mm
- net GND: track 0.00 -> 12.7 mm
- net VCC: track 0.00 -> 7.62 mm
- net Net-(U2-Pad7): track 0.00 -> 7.62 mm
- net Net-(U2-Pad6): track 0.00 -> 7.62 mm
- net Net-(J1-Pad1): track 0.00 -> 7.62 mm
- net Net-(C4-Pad2): track 0.00 -> 7.62 mm
- net Net-(U2-Pad1): track 0.00 -> 5.08 mm
- net Net-(C3-Pad2): track 0.00 -> 5.08 mm
- net Net-(C3-Pad1): track 0.00 -> 5.08 mm
Other:
- board size 150 x 50 mm -> 160 x 104.4 mm

Commit message: pcb
Parts:
- moved U2 31.8 mm to (153.9, 81.5)
- moved J1 17.4 mm to (49.5, 84.1)
Routing:
- net (no net): track 2199.6 -> 1328.7 mm
- net GND: track 12.7 -> 0.00 mm
- net VCC: track 7.62 -> 0.00 mm
- net Net-(U2-Pad7): track 7.62 -> 0.00 mm
- net Net-(U2-Pad6): track 7.62 -> 0.00 mm
- net Net-(J1-Pad1): track 7.62 -> 0.00 mm
- net Net-(C4-Pad2): track 7.62 -> 0.00 mm
- net Net-(U2-Pad1): track 5.08 -> 0.00 mm
- net Net-(C3-Pad2): track 5.08 -> 0.00 mm
- net Net-(C3-Pad1): track 5.08 -> 0.00 mm
Other:
- board size 160 x 104.4 mm -> 150 x 50 mm

Commit message: f proto2
Parts:
- J1: value Conn_01x02 -> Entrée Signal
- J2: value Conn_01x02 -> Sortie uControl
- J3: value Conn_01x02 -> Alim5V
- R1, R2: footprint Connector_PinSocket_2.54mm:PinSocket_1x06_P2.54mm_Vertical -> Resistor_THT:R_Axial_DIN0309_L9.0mm_D3.2mm_P12.70mm_Horizontal
- U1: value LM348D -> TL074
- moved C4 177.2 mm to (162.5, -72.9), turned to 180 degrees
- moved J3 161.8 mm to (119.6, -72.9)
- moved J1 160.7 mm to (84.1, -72.9), turned to 0 degrees
- moved U2 143.0 mm to (134.9, -60.2)
- moved C3 128.4 mm to (137.5, -55.1)
- moved R1 112.3 mm to (94.2, -39.9), turned to 180 degrees
- moved RV1 111.6 mm to (89.2, -45.0), turned to 90 degrees
- moved R2 109.5 mm to (145.0, -39.9), turned to 180 degrees
- moved U1 109.4 mm to (91.7, -50.0), turned to 90 degrees
- moved C2 109.1 mm to (112.0, -50.0)
- moved J2 103.9 mm to (165.4, -50.0), turned to 90 degrees
- moved RV2 97.0 mm to (137.4, -45.0), turned to 270 degrees
- moved C1 86.1 mm to (99.3, -34.8)
Connections:
- U1 pad 11: (no net) -> Net-(C4-Pad2)
- U1 pad 4: Net-(C4-Pad2) -> VCC
- U1 pad 8: VCC -> (no net)
Routing:
- net VCC: track 0.00 -> 7.62 mm
- net (no net): track 1328.7 -> 1321.1 mm
Other:
- board outline removed
