File: firstProto2/kicad/ampStation.kicad_pcb (KiCad board)
At the start: 2 copper layers, 13 parts, among them J1 Entrée Signal, J2 Sortie uControl, J3 Alim5V, U1 TL074, U2 MAX1044

Commit message: f proto2
Parts:
- moved J1 111.4 mm to (78.7, 38.4)
- moved J2 89.7 mm to (149.9, 38.4), turned to 0 degrees
- moved RV2 77.6 mm to (142.2, 32.5)
- moved RV1 75.7 mm to (88.9, 30.7)
- moved J3 75.4 mm to (94.0, -2.03)
- moved C4 74.1 mm to (157.2, 1.02)
- moved U1 73.2 mm to (91.4, 23.1)
- moved C2 72.9 mm to (114.3, 22.9)
- moved U2 71.8 mm to (121.9, 10.4)
- moved C3 71.3 mm to (124.5, 15.0)
- moved C1 68.5 mm to (111.8, 32.5)
- moved R2 68.2 mm to (149.9, 28.2)
- moved R1 66.3 mm to (94.0, 26.4)
Routing:
- net (no net): track 1321.1 -> 635.0 mm
- net GND: track 0.00 -> 587.0 mm
- net VCC: track 7.62 -> 132.7 mm, vias 0 -> 3
- net Net-(C4-Pad2): track 0.00 -> 75.0 mm, vias 0 -> 2
- net Net-(C1-Pad1): track 0.00 -> 63.9 mm
- net Net-(C2-Pad2): track 0.00 -> 45.3 mm, vias 0 -> 2
- net Net-(C3-Pad2): track 0.00 -> 26.4 mm
- net Net-(J1-Pad1): track 0.00 -> 18.8 mm
- net Net-(R1-Pad1): track 0.00 -> 10.2 mm
- net Net-(U2-Pad7): track 0.00 -> 7.62 mm
- net Net-(U2-Pad6): track 0.00 -> 7.62 mm
- net Net-(U2-Pad1): track 0.00 -> 5.08 mm
- net Net-(C3-Pad1): track 0.00 -> 5.08 mm
